Commit message: Move RealSense to front bumper mount, fix teleop and launch cleanup
- Add front_camera_mount on front bumper for clear forward camera view
- Fix use_stamped_vel: true for Jazzy diff_drive_controller compatibility
- Add pre-launch cleanup to kill zombie processes from previous runs
- Update RViz config with proper depth image normalization (0-10m range)
- Remove unused linter test files

Co-Authored-By: Claude Opus 4.6 <noreply@anthropic.com>

File: src/warebot/description/robot.urdf.xacro (robot description, xacro)
@@ -52,7 +52,7 @@
     <origin xyz="0.0 0.0 0.0" rpy="0.0 0.0 0.0"/>
   </xacro:velodyne_lidar>
-  <!-- Intel RealSense D435 depth camera on center of top plate -->
+  <!-- Intel RealSense D435 depth camera on front of robot -->
   <xacro:include filename="$(find clearpath_sensors_description)/urdf/intel_realsense.urdf.xacro"/>
-  <xacro:intel_realsense name="realsense" parent_link="top_plate_default_mount" model="d435">
+  <xacro:intel_realsense name="realsense" parent_link="front_camera_mount" model="d435">
     <origin xyz="0.0 0.0 0.0" rpy="0.0 0.0 0.0"/>
   </xacro:intel_realsense>
@@ -60,3 +60,10 @@
   <!-- Custom Links and Mounts                   -->
   <!-- ========================================= -->
+  <!-- Front camera mount on the front bumper -->
+  <link name="front_camera_mount"/>
+  <joint name="front_camera_mount_joint" type="fixed">
+    <parent link="front_bumper_mount"/>
+    <child link="front_camera_mount"/>
+    <origin xyz="0.0 0.0 0.05" rpy="0 0 0"/>
+  </joint>
 </robot>
